Commit message: Final Draft Version of Smoke_Bot

File: description/gazebo_control.xacro (robot description, xacro)
@@ -3,13 +3,11 @@
     <gazebo>
         <plugin name="diff_drive" filename="libgazebo_ros_diff_drive.so">
-            <!-- Wheel Information -->
             <left_joint>left_wheel_joint</left_joint>
             <right_joint>right_wheel_joint</right_joint>
-            <wheel_separation>0.15</wheel_separation>
-            <wheel_diameter>0.065</wheel_diameter>
+            <wheel_separation>0.55</wheel_separation>
+            <wheel_diameter>0.1</wheel_diameter>
             <!-- Limits -->
             <max_wheel_torque>200</max_wheel_torque>
             <max_wheel_acceleration>10.0</max_wheel_acceleration>
-            <!-- Output -->
             <odometry_frame>odom</odometry_frame>
             <robot_base_frame>base_link</robot_base_frame>

File: description/robot_core.xacro (robot description, xacro)
@@ -1,20 +1,37 @@
 <?xml version="1.0"?>
 <robot xmlns:xacro="http://www.ros.org/wiki/xacro" >
-   <xacro:include filename="inertial_macros.xacro"/>
-   <material name="white">
-       <color rgba="1 1 1 1" />
-   </material>
-   <material name="orange">
-       <color rgba="1 0.3 0.1 1"/>
-   </material>
-   <material name="blue">
-       <color rgba="0.2 0.2 1 1"/>
-   </material>
-   <material name="black">
-       <color rgba="0 0 0 1"/>
-   </material>
-   <link name="base_link">
-   </link>
-   <joint name="base_footprint_joint" type="fixed">
+    <xacro:include filename="inertial_macros.xacro"/>
+    <xacro:property name="chassis_length" value="0.65"/>
+    <xacro:property name="chassis_width" value="0.55"/>
+    <xacro:property name="chassis_height" value="0.138"/>
+    <xacro:property name="chassis_mass" value="1.0"/>
+    <xacro:property name="wheel_radius" value="0.1"/>
+    <xacro:property name="wheel_thickness" value="0.05"/>
+    <xacro:property name="wheel_mass" value="0.05"/>
+    <xacro:property name="wheel_offset_x" value="0.326"/>
+    <xacro:property name="wheel_offset_y" value="0.2785"/>
+    <xacro:property name="wheel_offset_z" value="0.01"/>
+    <xacro:property name="caster_wheel_radius" value="0.05"/>
+    <xacro:property name="caster_wheel_mass" value="0.01"/>
+    <xacro:property name="caster_wheel_offset_x" value="0.075"/>
+    <xacro:property name="caster_wheel_offset_z" value="${wheel_offset_z - wheel_radius + caster_wheel_radius}"/>
+    <material name="white">
+        <color rgba="1 1 1 1" />
+    </material>
+    <material name="orange">
+        <color rgba="1 0.3 0.1 1"/>
+    </material>
+    <material name="blue">
+        <color rgba="0.2 0.2 1 1"/>
+    </material>
+    <material name="black">
+        <color rgba="0 0 0 1"/>
+    </material>
+    <material name="red">
+        <color rgba="1 0 0 1"/>
+    </material>
+    <link name="base_link">
+    </link>
+    <joint name="base_footprint_joint" type="fixed">
         <parent link="base_link"/>
         <child link="base_footprint"/>
@@ -23,91 +40,105 @@
     <link name="base_footprint">
     </link>
-   <joint name="chassis_joint" type="fixed">
-       <parent link="base_link"/>
-       <child link="chassis"/>
-       <origin xyz="-0.1 0 0"/>
-   </joint>
-   <link name="chassis">
-       <visual>
-           <origin xyz="0.075 0 0.0025"/>
-           <geometry>
-               <box size="0.15 0.15 0.005"/>
-           </geometry>
-           <material name="white"/>
-       </visual>
-       <collision>
-           <origin xyz="0.075 0 0.0025"/>
-           <geometry>
-               <box size="0.15 0.15 0.0025"/>
-           </geometry>
-       </collision>
-       <xacro:inertial_box mass="0.5" x="0.15" y="0.15" z="0.005">
-           <origin xyz="0.075 0 0.0025" rpy="0 0 0"/>
-       </xacro:inertial_box>
-   </link>
-   <joint name="left_wheel_joint" type="continuous">
-       <parent link="base_link"/>
-       <child link="left_wheel"/>
-       <origin xyz="0 0.09 0" rpy="-${pi/2} 0 0" />
-       <axis xyz="0 0 1"/>
-   </joint>
-   <link name="left_wheel">
-       <visual>
-           <geometry>
-               <cylinder radius="0.0325" length="0.03"/>
-           </geometry>
-           <material name="blue"/>
-       </visual>
-       <collision>
-           <geometry>
-               <cylinder radius="0.0325" length="0.03"/>
-           </geometry>
-       </collision>
-       <xacro:inertial_cylinder mass="0.1" length="0.03" radius="0.0325">
-           <origin xyz="0 0 0" rpy="0 0 0"/>
-       </xacro:inertial_cylinder>
-   </link>
-   <joint name="right_wheel_joint" type="continuous">
-       <parent link="base_link"/>
-       <child link="right_wheel"/>
-       <origin xyz="0 -0.09 0" rpy="${pi/2} 0 0" />
-       <axis xyz="0 0 -1"/>
-   </joint>
-   <link name="right_wheel">
-       <visual>
-           <geometry>
-               <cylinder radius="0.0325" length="0.03"/>
-           </geometry>
-           <material name="blue"/>
-       </visual>
-       <collision>
-           <geometry>
-               <cylinder radius="0.0325" length="0.03"/>
-           </geometry>
-       </collision>
-       <xacro:inertial_cylinder mass="0.1" length="0.03" radius="0.0325">
-           <origin xyz="0 0 0" rpy="0 0 0"/>
-       </xacro:inertial_cylinder>
-   </link>
-   <joint name="caster_wheel_joint" type="fixed">
-       <parent link="chassis"/>
-       <child link="caster_wheel"/>
-       <origin xyz="0 0 0"/>
-   </joint>
-   <link name="caster_wheel">
-       <visual>
-           <geometry>
-               <sphere radius="0.03"/>
-           </geometry>
-           <material name="black"/>
-       </visual>
-       <collision>
-           <geometry>
-               <sphere radius="0.03"/>
-           </geometry>
-       </collision>
-       <xacro:inertial_sphere mass="0.1" radius="0.03">
-           <origin xyz="0 0 0" rpy="0 0 0"/>
-       </xacro:inertial_sphere>
-   </link>
+    <joint name="chassis_joint" type="fixed">
+        <parent link="base_link"/>
+        <child link="chassis"/>
+        <origin xyz="${-wheel_offset_x} 0 ${-wheel_offset_z}"/>
+    </joint>
+    <link name="chassis">
+        <visual>
+            <origin xyz="${chassis_length/2} 0 ${chassis_height/2}"/>
+            <geometry>
+                <box size="${chassis_length} ${chassis_width} ${chassis_height}"/>
+            </geometry>
+            <material name="orange"/>
+        </visual>
+        <collision>
+            <origin xyz="${chassis_length/2} 0 ${chassis_height/2}"/>
+            <geometry>
+                <box size="${chassis_length} ${chassis_width} ${chassis_height}"/>
+            </geometry>
+        </collision>
+        <xacro:inertial_box mass="0.5" x="${chassis_length}" y="${chassis_width}" z="${chassis_height}">
+            <origin xyz="${chassis_length/2} 0 ${chassis_height/2}" rpy="0 0 0"/>
+        </xacro:inertial_box>
+    </link>
+    <gazebo reference="chassis">
+        <material>Gazebo/Orange</material>
+    </gazebo>
+    <joint name="left_wheel_joint" type="continuous">
+        <parent link="base_link"/>
+        <child link="left_wheel"/>
+        <origin xyz="0 ${wheel_offset_y} 0" rpy="-${pi/2} 0 0" />
+        <axis xyz="0 0 1"/>
+    </joint>
+    <link name="left_wheel">
+        <visual>
+            <geometry>
+                <cylinder radius="${wheel_radius}" length="${wheel_thickness}"/>
+            </geometry>
+            <material name="blue"/>
+        </visual>
+        <collision>
+            <geometry>
+                <sphere radius="${wheel_radius}"/>
+            </geometry>
+        </collision>
+        <xacro:inertial_cylinder mass="${wheel_mass}" length="${wheel_thickness}" radius="${wheel_radius}">
+            <origin xyz="0 0 0" rpy="0 0 0"/>
+        </xacro:inertial_cylinder>
+    </link>
+    <gazebo reference="left_wheel">
+        <material>Gazebo/Blue</material>
+    </gazebo>
+    <joint name="right_wheel_joint" type="continuous">
+        <parent link="base_link"/>
+        <child link="right_wheel"/>
+        <origin xyz="0 ${-wheel_offset_y} 0" rpy="${pi/2} 0 0" />
+        <axis xyz="0 0 -1"/>
+    </joint>
+    <link name="right_wheel">
+        <visual>
+            <geometry>
+                <cylinder radius="${wheel_radius}" length="${wheel_thickness}"/>
+            </geometry>
+            <material name="blue"/>
+        </visual>
+        <collision>
+            <geometry>
+                <sphere radius="${wheel_radius}"/>
+            </geometry>
+        </collision>
+        <xacro:inertial_cylinder mass="${wheel_mass}" length="${wheel_thickness}" radius="${wheel_radius}">
+            <origin xyz="0 0 0" rpy="0 0 0"/>
+        </xacro:inertial_cylinder>
+    </link>
+    <gazebo reference="right_wheel">
+        <material>Gazebo/Blue</material>
+    </gazebo>
+    <joint name="caster_wheel_joint" type="fixed">
+        <parent link="chassis"/>
+        <child link="caster_wheel"/>
+        <origin xyz="${caster_wheel_offset_x} 0 ${caster_wheel_offset_z}"/>
+    </joint>
+    <link name="caster_wheel">
+        <visual>
+            <geometry>
+                <sphere radius="${caster_wheel_radius}"/>
+            </geometry>
+            <material name="white"/>
+        </visual>
+        <collision>
+            <geometry>
+                <sphere radius="${caster_wheel_radius}"/>
+            </geometry>
+        </collision>
+        <xacro:inertial_sphere mass="${caster_wheel_mass}" radius="${caster_wheel_radius}">
+            <origin xyz="0 0 0" rpy="0 0 0"/>
+        </xacro:inertial_sphere>
+    </link>
+    <gazebo reference="caster_wheel">
+        <material>Gazebo/White</material>
+        <mu1 value="0.001"/>
+        <mu2 value="0.001"/>
+    </gazebo>
 </robot>
